Commit message: Made changes to reflect new rl kit setup

File: spot_curobo_config/urdf/spot.urdf (robot description, URDF)
Before this commit: robot spot, 37 links, 36 joints
Links:
- removed link lidar_assembly
- added link alpha_detector_face
- added link alpha_detector_sensing_frame
- added link payload_mount_reference_frame
- added link rl_kit_gxp_interface; visual mesh filename=meshes/accessories/gxp.dae
- added link rl_kit_jetson_housing_box; collision box size=0.156 0.206 0.112; visual box size=0.156 0.206 0.112
- added link rl_kit_reference_frame
- added link rl_kit_velodyne_mounting_plate; collision box size=0.19 0.18 0.013; visual mesh filename=meshes/accessories/rl_kit_velodyne_mount.dae
- added link rl_kit_wire_housing_box; collision box size=0.152 0.206 0.066; visual box size=0.152 0.206 0.066
- added link velodyne_cage; collision cylinder length=0.08 radius=0.08; visual mesh filename=meshes/accessories/velodyne_cage.dae
- link arm0_elbow_pitch: geometry collision mesh filename=meshes/arm/arm0.link_el0.obj; visual mesh filename=meshes/arm/arm0.link_el0.dae
- link arm0_elbow_roll: geometry collision mesh filename=meshes/arm/arm0.link_el1.obj; visual mesh filename=meshes/arm/arm0.link_el1.dae
- link arm0_fingers: geometry collision mesh filename=meshes/arm/arm0.link_fngr.obj; visual mesh filename=meshes/arm/arm0.link_fngr.dae
- link arm0_shoulder_roll: geometry collision mesh filename=meshes/arm/arm0.link_hr0.obj; visual mesh filename=meshes/arm/arm0.link_hr0.dae
- link arm0_shoulder_yaw: geometry collision mesh filename=meshes/arm/arm0.link_sh0.obj; visual mesh filename=meshes/arm/arm0.link_sh0.dae
- link arm0_wrist_pitch: geometry collision mesh filename=meshes/arm/arm0.link_wr0.obj; visual mesh filename=meshes/arm/arm0.link_wr0.dae
- link arm0_wrist_roll: geometry collision mesh filename=meshes/arm/arm0.link_wr1.obj; visual mesh filename=meshes/arm/arm0.link_wr1.dae
Joints:
- removed joint lidar_mount
- added joint alpha_detector_joint: type fixed, parent arm0_hand, child alpha_detector_face, origin xyz=0.04 0.0 -0.03
- added joint alpha_detector_sensor_joint: type fixed, parent alpha_detector_face, child alpha_detector_sensing_frame, origin rpy=0.0 1.5707963267948966 0.0
- added joint payload_mount_reference_frame_joint: type fixed, parent base_link, child payload_mount_reference_frame, origin xyz=0.2075 0.0 0.0805
- added joint rl_kit_base_mount_to_body: type fixed, parent payload_mount_reference_frame, child rl_kit_reference_frame, origin xyz=-0.292 0.0 0.056
- added joint rl_kit_gxp_joint: type fixed, parent rl_kit_reference_frame, child rl_kit_gxp_interface, origin xyz=0.13 0.0 -0.056
- added joint rl_kit_jetson_housing_box_joint: type fixed, parent rl_kit_reference_frame, child rl_kit_jetson_housing_box, origin xyz=-0.078 0.0 0.0
- added joint rl_kit_velodyne_mount_joint: type fixed, parent rl_kit_jetson_housing_box, child rl_kit_velodyne_mounting_plate, origin xyz=-0.045 0.0 0.056
- added joint rl_kit_wire_housing_box_joint: type fixed, parent rl_kit_reference_frame, child rl_kit_wire_housing_box, origin xyz=0.076 0.0 -0.023
- added joint velodyne_cage_link: type fixed, parent rl_kit_velodyne_mounting_plate, child velodyne_cage, origin xyz=0 0 0.0065
- joint velodyne_base_mount_joint: origin xyz=0.0 0 0.08 rpy=0 0 0 -> xyz=0 0 0.008 rpy=0 0 0; parent lidar_assembly -> rl_kit_velodyne_mounting_plate
