Commit message: Added more collision exclusions that will never happen to increase planning efficiency

File: spot_moveit_config/config/accessories/rl_kit.srdf.xacro (robot description, xacro)
@@ -1,25 +1,43 @@
 <?xml version="1.0" encoding="UTF-8"?>
 <robot name="rl_kit_srdf" xmlns:xacro="http://www.ros.org/wiki/xacro">
-    <disable_collisions link1="arm0_base_link" link2="rl_kit_jetson_housing_box" reason="Adjacent"/>
-    <disable_collisions link1="arm0_base_link" link2="rl_kit_wire_housing_box" reason="Adjacent"/>
+    <disable_collisions link1="arm0_base_link" link2="rl_kit_jetson_housing_box" reason="Never"/>
+    <disable_collisions link1="arm0_base_link" link2="rl_kit_wire_housing_box" reason="Never"/>
+    <disable_collisions link1="arm0_base_link" link2="rl_kit_gxp_interface" reason="Never"/>
     <disable_collisions link1="arm0_shoulder_pitch" link2="rl_kit_jetson_housing_box" reason="Never"/>
     <disable_collisions link1="arm0_shoulder_pitch" link2="rl_kit_wire_housing_box" reason="Never"/>
+    <disable_collisions link1="arm0_shoulder_pitch" link2="rl_kit_gxp_interface" reason="Never"/>
     <disable_collisions link1="arm0_shoulder_roll" link2="rl_kit_jetson_housing_box" reason="Never"/>
     <disable_collisions link1="arm0_shoulder_yaw" link2="rl_kit_jetson_housing_box" reason="Never"/>
+    <disable_collisions link1="arm0_shoulder_yaw" link2="rl_kit_gxp_interface" reason="Never"/>
     <disable_collisions link1="arm0_shoulder_yaw" link2="rl_kit_wire_housing_box" reason="Never"/>
     <disable_collisions link1="body" link2="rl_kit_jetson_housing_box" reason="Adjacent"/>
     <disable_collisions link1="body" link2="rl_kit_wire_housing_box" reason="Adjacent"/>
+    <disable_collisions link1="body" link2="rl_kit_gxp_interface" reason="Adjacent"/>
     <disable_collisions link1="front_left_hip" link2="rl_kit_jetson_housing_box" reason="Never"/>
     <disable_collisions link1="front_left_hip" link2="rl_kit_wire_housing_box" reason="Never"/>
+    <disable_collisions link1="front_left_hip" link2="rl_kit_gxp_interface" reason="Never"/>
     <disable_collisions link1="front_left_upper_leg" link2="rl_kit_jetson_housing_box" reason="Never"/>
+    <disable_collisions link1="front_left_upper_leg" link2="rl_kit_wire_housing_box" reason="Never"/>
+    <disable_collisions link1="front_left_upper_leg" link2="rl_kit_gxp_interface" reason="Never"/>
     <disable_collisions link1="front_right_hip" link2="rl_kit_jetson_housing_box" reason="Never"/>
     <disable_collisions link1="front_right_hip" link2="rl_kit_wire_housing_box" reason="Never"/>
+    <disable_collisions link1="front_right_hip" link2="rl_kit_gxp_interface" reason="Never"/>
     <disable_collisions link1="front_right_upper_leg" link2="rl_kit_jetson_housing_box" reason="Never"/>
+    <disable_collisions link1="front_right_upper_leg" link2="rl_kit_wire_housing_box" reason="Never"/>
+    <disable_collisions link1="front_right_upper_leg" link2="rl_kit_gxp_interface" reason="Never"/>
     <disable_collisions link1="rear_left_hip" link2="rl_kit_jetson_housing_box" reason="Never"/>
     <disable_collisions link1="rear_left_hip" link2="rl_kit_wire_housing_box" reason="Never"/>
+    <disable_collisions link1="rear_left_hip" link2="rl_kit_gxp_interface" reason="Never"/>
+    <disable_collisions link1="rear_left_upper_leg" link2="rl_kit_jetson_housing_box" reason="Never"/>
     <disable_collisions link1="rear_left_upper_leg" link2="rl_kit_wire_housing_box" reason="Never"/>
+    <disable_collisions link1="rear_left_upper_leg" link2="rl_kit_gxp_interface" reason="Never"/>
     <disable_collisions link1="rear_right_hip" link2="rl_kit_jetson_housing_box" reason="Never"/>
     <disable_collisions link1="rear_right_hip" link2="rl_kit_wire_housing_box" reason="Never"/>
+    <disable_collisions link1="rear_right_hip" link2="rl_kit_gxp_interface" reason="Never"/>
+    <disable_collisions link1="rear_right_upper_leg" link2="rl_kit_jetson_housing_box" reason="Never"/>
     <disable_collisions link1="rear_right_upper_leg" link2="rl_kit_wire_housing_box" reason="Never"/>
+    <disable_collisions link1="rear_right_upper_leg" link2="rl_kit_gxp_interface" reason="Never"/>
     <disable_collisions link1="rl_kit_jetson_housing_box" link2="rl_kit_wire_housing_box" reason="Adjacent"/>
+    <disable_collisions link1="rl_kit_jetson_housing_box" link2="rl_kit_gxp_interface" reason="Never"/>
+    <disable_collisions link1="rl_kit_wire_housing_box" link2="rl_kit_gxp_interface" reason="Never"/>
 </robot>
