Commit message: moves on spot but move group dies; trying to remove extraneous joints

File: spot_moveit_config/config/spot.ros2_control.xacro (robot description, xacro)
@@ -8,29 +8,6 @@
                 <plugin>mock_components/GenericSystem</plugin>
             </hardware>
-            <joint name="body_height_joint">
-                <state_interface name="position">
-                  <param name="initial_value">${initial_positions['body_height_joint']}</param>
-                </state_interface>
-                <state_interface name="velocity"/>
-            </joint>
-            <joint name="body_yaw_joint">
-                <state_interface name="position">
-                  <param name="initial_value">${initial_positions['body_yaw_joint']}</param>
-                </state_interface>
-                <state_interface name="velocity"/>
-            </joint>
-            <joint name="body_pitch_joint">
-                <state_interface name="position">
-                  <param name="initial_value">${initial_positions['body_pitch_joint']}</param>
-                </state_interface>
-                <state_interface name="velocity"/>
-            </joint>
-            <joint name="body_roll_joint">
-                <state_interface name="position">
-                  <param name="initial_value">${initial_positions['body_roll_joint']}</param>
-                </state_interface>
-                <state_interface name="velocity"/>
-            </joint>
             <joint name="arm0_shoulder_yaw">
+                <command_interface name="position"/>
                 <state_interface name="position">
                   <param name="initial_value">${initial_positions['arm0_shoulder_yaw']}</param>
@@ -39,4 +16,5 @@
             </joint>
             <joint name="arm0_shoulder_pitch">
+                <command_interface name="position"/>
                 <state_interface name="position">
                   <param name="initial_value">${initial_positions['arm0_shoulder_pitch']}</param>
@@ -45,4 +23,5 @@
             </joint>
             <joint name="arm0_elbow_pitch">
+                <command_interface name="position"/>
                 <state_interface name="position">
                   <param name="initial_value">${initial_positions['arm0_elbow_pitch']}</param>
@@ -51,4 +30,5 @@
             </joint>
             <joint name="arm0_elbow_roll">
+                <command_interface name="position"/>
                 <state_interface name="position">
                   <param name="initial_value">${initial_positions['arm0_elbow_roll']}</param>
@@ -57,4 +37,5 @@
             </joint>
             <joint name="arm0_wrist_pitch">
+                <command_interface name="position"/>
                 <state_interface name="position">
                   <param name="initial_value">${initial_positions['arm0_wrist_pitch']}</param>
@@ -63,4 +44,5 @@
             </joint>
             <joint name="arm0_wrist_roll">
+                <command_interface name="position"/>
                 <state_interface name="position">
                   <param name="initial_value">${initial_positions['arm0_wrist_roll']}</param>

File: spot_moveit_config/config/spot.urdf.xacro (robot description, xacro)
@@ -3,5 +3,5 @@
     <xacro:arg name="initial_positions_file" default="initial_positions.yaml" />
     <!-- Import spot urdf file -->
-    <xacro:include filename="$(find spot_description)/urdf/spot.urdf.xacro" />
+    <xacro:include filename="$(find spot_description)/urdf/spot_with_arm.urdf.xacro" />
     <!-- Import control_xacro -->
     <xacro:include filename="spot.ros2_control.xacro" />

Commit message: Added a launch fiel for running a virtual controller with Spot config

File: spot_moveit_config/config/spot.ros2_control.xacro (robot description, xacro)
@@ -2,4 +2,5 @@
 <robot xmlns:xacro="http://www.ros.org/wiki/xacro">
     <xacro:macro name="spot_ros2_control" params="name initial_positions_file">
+        <xacro:arg name="kinematic_model" default="none"/>
         <xacro:property name="initial_positions" value="${load_yaml(initial_positions_file)['initial_positions']}"/>
         <ros2_control name="${name}" type="system">
@@ -8,29 +9,36 @@
                 <plugin>mock_components/GenericSystem</plugin>
             </hardware>
-            <joint name="body_height_joint">
-                <state_interface name="position">
-                  <param name="initial_value">${initial_positions['body_height_joint']}</param>
-                </state_interface>
-                <state_interface name="velocity"/>
-            </joint>
-            <joint name="body_yaw_joint">
-                <state_interface name="position">
-                  <param name="initial_value">${initial_positions['body_yaw_joint']}</param>
-                </state_interface>
-                <state_interface name="velocity"/>
-            </joint>
-            <joint name="body_pitch_joint">
-                <state_interface name="position">
-                  <param name="initial_value">${initial_positions['body_pitch_joint']}</param>
-                </state_interface>
-                <state_interface name="velocity"/>
-            </joint>
-            <joint name="body_roll_joint">
-                <state_interface name="position">
-                  <param name="initial_value">${initial_positions['body_roll_joint']}</param>
-                </state_interface>
-                <state_interface name="velocity"/>
-            </joint>
+            <xacro:if value="${kinematic_model == 'body_assist'}">
+              <joint name="body_height_joint">
+                  <command_interface name="position"/>
+                  <state_interface name="position">
+                    <param name="initial_value">${initial_positions['body_height_joint']}</param>
+                  </state_interface>
+                  <state_interface name="velocity"/>
+              </joint>
+              <joint name="body_yaw_joint">
+                  <command_interface name="position"/>
+                  <state_interface name="position">
+                    <param name="initial_value">${initial_positions['body_yaw_joint']}</param>
+                  </state_interface>
+                  <state_interface name="velocity"/>
+              </joint>
+              <joint name="body_pitch_joint">
+                  <command_interface name="position"/>
+                  <state_interface name="position">
+                    <param name="initial_value">${initial_positions['body_pitch_joint']}</param>
+                  </state_interface>
+                  <state_interface name="velocity"/>
+              </joint>
+              <joint name="body_roll_joint">
+                  <command_interface name="position"/>
+                  <state_interface name="position">
+                    <param name="initial_value">${initial_positions['body_roll_joint']}</param>
+                  </state_interface>
+                  <state_interface name="velocity"/>
+              </joint>
+            </xacro:if>
             <joint name="arm0_shoulder_yaw">
+                <command_interface name="position"/>
                 <state_interface name="position">
                   <param name="initial_value">${initial_positions['arm0_shoulder_yaw']}</param>
@@ -39,4 +47,5 @@
             </joint>
             <joint name="arm0_shoulder_pitch">
+                <command_interface name="position"/>
                 <state_interface name="position">
                   <param name="initial_value">${initial_positions['arm0_shoulder_pitch']}</param>
@@ -45,4 +54,5 @@
             </joint>
             <joint name="arm0_elbow_pitch">
+                <command_interface name="position"/>
                 <state_interface name="position">
                   <param name="initial_value">${initial_positions['arm0_elbow_pitch']}</param>
@@ -51,4 +61,5 @@
             </joint>
             <joint name="arm0_elbow_roll">
+                <command_interface name="position"/>
                 <state_interface name="position">
                   <param name="initial_value">${initial_positions['arm0_elbow_roll']}</param>
@@ -57,4 +68,5 @@
             </joint>
             <joint name="arm0_wrist_pitch">
+                <command_interface name="position"/>
                 <state_interface name="position">
                   <param name="initial_value">${initial_positions['arm0_wrist_pitch']}</param>
@@ -63,4 +75,5 @@
             </joint>
             <joint name="arm0_wrist_roll">
+                <command_interface name="position"/>
                 <state_interface name="position">
                   <param name="initial_value">${initial_positions['arm0_wrist_roll']}</param>

Commit message: Cleaned up ros2 xacro and added all remaining non-controller joint positions to visualization

File: spot_moveit_config/config/spot.ros2_control.xacro (robot description, xacro)
@@ -9,76 +9,48 @@
                 <plugin>mock_components/GenericSystem</plugin>
             </hardware>
+            <!-- Controlled joints -->
+            <xacro:macro name="AddControlledJoint" params="joint_name">
+                <joint name="${joint_name}">
+                    <command_interface name="position"/>
+                    <state_interface name="position">
+                        <param name="initial_value">${initial_positions[joint_name]}</param>
+                    </state_interface>
+                    <state_interface name="velocity"/>"
+                </joint>
+            </xacro:macro>
             <xacro:if value="${kinematic_model == 'body_assist'}">
-              <joint name="body_height_joint">
-                  <command_interface name="position"/>
-                  <state_interface name="position">
-                    <param name="initial_value">${initial_positions['body_height_joint']}</param>
-                  </state_interface>
-                  <state_interface name="velocity"/>
-              </joint>
-              <joint name="body_yaw_joint">
-                  <command_interface name="position"/>
-                  <state_interface name="position">
-                    <param name="initial_value">${initial_positions['body_yaw_joint']}</param>
-                  </state_interface>
-                  <state_interface name="velocity"/>
-              </joint>
-              <joint name="body_pitch_joint">
-                  <command_interface name="position"/>
-                  <state_interface name="position">
-                    <param name="initial_value">${initial_positions['body_pitch_joint']}</param>
-                  </state_interface>
-                  <state_interface name="velocity"/>
-              </joint>
-              <joint name="body_roll_joint">
-                  <command_interface name="position"/>
-                  <state_interface name="position">
-                    <param name="initial_value">${initial_positions['body_roll_joint']}</param>
-                  </state_interface>
-                  <state_interface name="velocity"/>
-              </joint>
+                <xacro:AddControlledJoint joint_name="body_height_joint"/>
+                <xacro:AddControlledJoint joint_name="body_yaw_joint"/>
+                <xacro:AddControlledJoint joint_name="body_pitch_joint"/>
+                <xacro:AddControlledJoint joint_name="body_roll_joint"/>
             </xacro:if>
-            <joint name="arm0_shoulder_yaw">
-                <command_interface name="position"/>
-                <state_interface name="position">
-                  <param name="initial_value">${initial_positions['arm0_shoulder_yaw']}</param>
-                </state_interface>
-                <state_interface name="velocity"/>
-            </joint>
-            <joint name="arm0_shoulder_pitch">
-                <command_interface name="position"/>
-                <state_interface name="position">
-                  <param name="initial_value">${initial_positions['arm0_shoulder_pitch']}</param>
-                </state_interface>
-                <state_interface name="velocity"/>
-            </joint>
-            <joint name="arm0_elbow_pitch">
-                <command_interface name="position"/>
-                <state_interface name="position">
-                  <param name="initial_value">${initial_positions['arm0_elbow_pitch']}</param>
-                </state_interface>
-                <state_interface name="velocity"/>
-            </joint>
-            <joint name="arm0_elbow_roll">
-                <command_interface name="position"/>
-                <state_interface name="position">
-                  <param name="initial_value">${initial_positions['arm0_elbow_roll']}</param>
-                </state_interface>
-                <state_interface name="velocity"/>
-            </joint>
-            <joint name="arm0_wrist_pitch">
-                <command_interface name="position"/>
-                <state_interface name="position">
-                  <param name="initial_value">${initial_positions['arm0_wrist_pitch']}</param>
-                </state_interface>
-                <state_interface name="velocity"/>
-            </joint>
-            <joint name="arm0_wrist_roll">
-                <command_interface name="position"/>
-                <state_interface name="position">
-                  <param name="initial_value">${initial_positions['arm0_wrist_roll']}</param>
-                </state_interface>
-                <state_interface name="velocity"/>
-            </joint>
+            <xacro:AddControlledJoint joint_name="arm0_shoulder_yaw"/>
+            <xacro:AddControlledJoint joint_name="arm0_shoulder_pitch"/>
+            <xacro:AddControlledJoint joint_name="arm0_elbow_pitch"/>
+            <xacro:AddControlledJoint joint_name="arm0_elbow_roll"/>
+            <xacro:AddControlledJoint joint_name="arm0_wrist_pitch"/>
+            <xacro:AddControlledJoint joint_name="arm0_wrist_roll"/>
+            <!-- Non-controlled joints -->
+            <xacro:macro name="AddNonControlledJoint" params="joint_name">
+                <joint name="${joint_name}">
+                    <state_interface name="position">
+                        <param name="initial_value">${initial_positions[joint_name]}</param>
+                    </state_interface>
+                    <state_interface name="velocity"/>"
+                </joint>
+            </xacro:macro>
+            <xacro:AddNonControlledJoint joint_name="front_left_hip_x"/>
+            <xacro:AddNonControlledJoint joint_name="front_left_hip_y"/>
+            <xacro:AddNonControlledJoint joint_name="front_left_knee"/>
+            <xacro:AddNonControlledJoint joint_name="front_right_hip_x"/>
+            <xacro:AddNonControlledJoint joint_name="front_right_hip_y"/>
+            <xacro:AddNonControlledJoint joint_name="front_right_knee"/>
+            <xacro:AddNonControlledJoint joint_name="rear_left_hip_x"/>
+            <xacro:AddNonControlledJoint joint_name="rear_left_hip_y"/>
+            <xacro:AddNonControlledJoint joint_name="rear_left_knee"/>
+            <xacro:AddNonControlledJoint joint_name="rear_right_hip_x"/>
+            <xacro:AddNonControlledJoint joint_name="rear_right_hip_y"/>
+            <xacro:AddNonControlledJoint joint_name="rear_right_knee"/>
+            <xacro:AddNonControlledJoint joint_name="arm0_fingers"/>
         </ros2_control>
     </xacro:macro>

Commit message: add topic-based ros2_control plugin

File: spot_moveit_config/config/spot.ros2_control.xacro (robot description, xacro)
@@ -1,11 +1,17 @@
 <?xml version="1.0"?>
 <robot xmlns:xacro="http://www.ros.org/wiki/xacro">
-    <xacro:macro name="spot_ros2_control" params="name initial_positions_file">
+    <xacro:macro name="spot_ros2_control" params="name initial_positions_file ros2_control_hardware_type">
         <xacro:arg name="kinematic_model" default="none"/>
         <xacro:property name="initial_positions" value="${load_yaml(initial_positions_file)['initial_positions']}"/>
         <ros2_control name="${name}" type="system">
             <hardware>
-                <!-- By default, set up controllers for simulation. This won't work on real hardware -->
-                <plugin>mock_components/GenericSystem</plugin>
+                <xacro:if value="${ros2_control_hardware_type == 'mock_components'}">
+                    <plugin>mock_components/GenericSystem</plugin>
+                </xacro:if>
+                <xacro:if value="${ros2_control_hardware_type == 'isaac'}">
+                    <plugin>topic_based_ros2_control/TopicBasedSystem</plugin>
+                    <param name="joint_commands_topic">/isaac_joint_commands</param>
+                    <param name="joint_states_topic">/isaac_joint_states</param>
+                </xacro:if>
             </hardware>
             <!-- Controlled joints -->

File: spot_moveit_config/config/spot.urdf.xacro (robot description, xacro)
@@ -2,8 +2,9 @@
 <robot xmlns:xacro="http://www.ros.org/wiki/xacro" name="spot">
     <xacro:arg name="initial_positions_file" default="initial_positions.yaml" />
+    <xacro:arg name="ros2_control_hardware_type" default="mock_components" />
     <!-- Import spot urdf file -->
     <xacro:include filename="$(find spot_description)/urdf/spot.urdf.xacro" />
     <!-- Import control_xacro -->
     <xacro:include filename="spot.ros2_control.xacro" />
-    <xacro:spot_ros2_control name="FakeSystem" initial_positions_file="$(arg initial_positions_file)"/>
+    <xacro:spot_ros2_control name="FakeSystem" initial_positions_file="$(arg initial_positions_file)" ros2_control_hardware_type="$(arg ros2_control_hardware_type)"/>
 </robot>
