Commit message: Removed leftover references to accessories in the main srdf xacro

File: spot_moveit_config/config/spot.srdf.xacro (robot description, xacro)
@@ -131,10 +131,6 @@
     <disable_collisions link1="rear_right_lower_leg" link2="rear_right_upper_leg" reason="Adjacent"/>
     <disable_collisions link1="rear_right_upper_leg" link2="velodyne_base_link" reason="Never"/>
-    <disable_collisions link1="body" link2="eap_2_assembly" reason="Adjacent"/>
     <disable_collisions link1="arm0_base_link" link2="arm0_shoulder_yaw" reason="Adjacent"/>
     <disable_collisions link1="arm0_base_link" link2="body" reason="Adjacent"/>
-    <disable_collisions link1="alpha_detector" link2="arm0_wrist_roll" reason="Adjacent"/>
-    <disable_collisions link1="alpha_detector" link2="arm0_wrist_pitch" reason="Adjacent"/>
-    <disable_collisions link1="alpha_detector" link2="arm0_fingers" reason="Adjacent"/>
     <!-- Accessory collisions -->
     <xacro:if value="$(arg has_eap)">

Commit message: Removed references to velodyne from the base srdf

File: spot_moveit_config/config/spot.srdf.xacro (robot description, xacro)
@@ -5,7 +5,4 @@
 -->
 <robot name="spot" xmlns:xacro="http://www.ros.org/wiki/xacro">
-    <xacro:arg name="has_eap"    default="False"/>
-    <xacro:arg name="has_eap_2"  default="False"/>
-    <xacro:arg name="has_rl_kit" default="False"/>
     <!--GROUPS: Representation of a set of joints and links. This can be useful for specifying DOF to plan for, defining arms, end effectors, etc-->
     <!--LINKS: When a link is specified, the parent joint of that link (if it exists) is automatically included-->
@@ -54,5 +51,4 @@
     <disable_collisions link1="arm0_shoulder_pitch" link2="rear_right_lower_leg" reason="Never"/>
     <disable_collisions link1="arm0_shoulder_pitch" link2="rear_right_upper_leg" reason="Never"/>
-    <disable_collisions link1="arm0_shoulder_pitch" link2="velodyne_base_link" reason="Never"/>
     <disable_collisions link1="arm0_shoulder_roll" link2="arm0_shoulder_yaw" reason="Default"/>
     <disable_collisions link1="arm0_shoulder_roll" link2="arm0_wrist_pitch" reason="Never"/>
@@ -63,5 +59,4 @@
     <disable_collisions link1="arm0_shoulder_roll" link2="rear_right_hip" reason="Never"/>
     <disable_collisions link1="arm0_shoulder_roll" link2="rear_right_upper_leg" reason="Never"/>
-    <disable_collisions link1="arm0_shoulder_roll" link2="velodyne_base_link" reason="Never"/>
     <disable_collisions link1="arm0_shoulder_yaw" link2="body" reason="Adjacent"/>
     <disable_collisions link1="arm0_shoulder_yaw" link2="front_left_hip" reason="Never"/>
@@ -73,5 +68,4 @@
     <disable_collisions link1="arm0_shoulder_yaw" link2="rear_right_lower_leg" reason="Never"/>
     <disable_collisions link1="arm0_shoulder_yaw" link2="rear_right_upper_leg" reason="Never"/>
-    <disable_collisions link1="arm0_shoulder_yaw" link2="velodyne_base_link" reason="Never"/>
     <disable_collisions link1="arm0_wrist_pitch" link2="arm0_wrist_roll" reason="Adjacent"/>
     <disable_collisions link1="body" link2="front_left_hip" reason="Adjacent"/>
@@ -83,5 +77,4 @@
     <disable_collisions link1="body" link2="rear_right_hip" reason="Adjacent"/>
     <disable_collisions link1="body" link2="rear_right_upper_leg" reason="Default"/>
-    <disable_collisions link1="body" link2="velodyne_base_link" reason="Never"/>
     <disable_collisions link1="front_left_hip" link2="front_left_lower_leg" reason="Never"/>
     <disable_collisions link1="front_left_hip" link2="front_left_upper_leg" reason="Adjacent"/>
@@ -93,5 +86,4 @@
     <disable_collisions link1="front_left_hip" link2="rear_right_lower_leg" reason="Never"/>
     <disable_collisions link1="front_left_hip" link2="rear_right_upper_leg" reason="Never"/>
-    <disable_collisions link1="front_left_hip" link2="velodyne_base_link" reason="Never"/>
     <disable_collisions link1="front_left_lower_leg" link2="front_left_upper_leg" reason="Adjacent"/>
     <disable_collisions link1="front_left_lower_leg" link2="front_right_hip" reason="Never"/>
@@ -101,5 +93,4 @@
     <disable_collisions link1="front_left_upper_leg" link2="rear_right_hip" reason="Never"/>
     <disable_collisions link1="front_left_upper_leg" link2="rear_right_upper_leg" reason="Never"/>
-    <disable_collisions link1="front_left_upper_leg" link2="velodyne_base_link" reason="Never"/>
     <disable_collisions link1="front_right_hip" link2="front_right_lower_leg" reason="Never"/>
     <disable_collisions link1="front_right_hip" link2="front_right_upper_leg" reason="Adjacent"/>
@@ -110,5 +101,4 @@
     <disable_collisions link1="front_right_hip" link2="rear_right_lower_leg" reason="Never"/>
     <disable_collisions link1="front_right_hip" link2="rear_right_upper_leg" reason="Never"/>
-    <disable_collisions link1="front_right_hip" link2="velodyne_base_link" reason="Never"/>
     <disable_collisions link1="front_right_lower_leg" link2="front_right_upper_leg" reason="Adjacent"/>
     <disable_collisions link1="front_right_lower_leg" link2="rear_left_hip" reason="Never"/>
@@ -116,22 +106,20 @@
     <disable_collisions link1="front_right_upper_leg" link2="rear_left_upper_leg" reason="Never"/>
     <disable_collisions link1="front_right_upper_leg" link2="rear_right_hip" reason="Never"/>
-    <disable_collisions link1="front_right_upper_leg" link2="velodyne_base_link" reason="Never"/>
     <disable_collisions link1="rear_left_hip" link2="rear_left_lower_leg" reason="Never"/>
     <disable_collisions link1="rear_left_hip" link2="rear_left_upper_leg" reason="Adjacent"/>
     <disable_collisions link1="rear_left_hip" link2="rear_right_lower_leg" reason="Never"/>
     <disable_collisions link1="rear_left_hip" link2="rear_right_upper_leg" reason="Never"/>
-    <disable_collisions link1="rear_left_hip" link2="velodyne_base_link" reason="Never"/>
     <disable_collisions link1="rear_left_lower_leg" link2="rear_left_upper_leg" reason="Adjacent"/>
     <disable_collisions link1="rear_left_lower_leg" link2="rear_right_hip" reason="Never"/>
     <disable_collisions link1="rear_left_upper_leg" link2="rear_right_hip" reason="Never"/>
-    <disable_collisions link1="rear_left_upper_leg" link2="velodyne_base_link" reason="Never"/>
     <disable_collisions link1="rear_right_hip" link2="rear_right_lower_leg" reason="Never"/>
     <disable_collisions link1="rear_right_hip" link2="rear_right_upper_leg" reason="Adjacent"/>
-    <disable_collisions link1="rear_right_hip" link2="velodyne_base_link" reason="Never"/>
     <disable_collisions link1="rear_right_lower_leg" link2="rear_right_upper_leg" reason="Adjacent"/>
-    <disable_collisions link1="rear_right_upper_leg" link2="velodyne_base_link" reason="Never"/>
     <disable_collisions link1="arm0_base_link" link2="arm0_shoulder_yaw" reason="Adjacent"/>
     <disable_collisions link1="arm0_base_link" link2="body" reason="Adjacent"/>
     <!-- Accessory collisions -->
+    <xacro:arg name="has_eap"    default="False"/>
+    <xacro:arg name="has_eap_2"  default="False"/>
+    <xacro:arg name="has_rl_kit" default="False"/>
     <xacro:if value="$(arg has_eap)">
         <xacro:include filename="$(find spot_moveit_config)/config/accessories/eap.srdf.xacro"/>

Commit message: Fixed moveit issues when kinematic model is 'none'

File: spot_moveit_config/config/spot.srdf.xacro (robot description, xacro)
@@ -10,15 +10,25 @@
     <!--CHAINS: When a chain is specified, all the links along the chain (including endpoints) are included in the group. Additionally, all the joints that are parents to included links are also included. This means that joints along the chain and the parent joint of the base link are included in the group-->
     <!--SUBGROUPS: Groups can also be formed by referencing to already defined group names-->
-    <group name="arm_with_body">
-        <chain base_link="base_footprint" tip_link="arm0_hand"/>
-    </group>
     <group name="arm">
         <chain base_link="arm0_base_link" tip_link="arm0_hand"/>
     </group>
+    <!-- Add the extra group if full body control is enabled -->
+    <xacro:arg name="kinematic_model" default="none"/>
+    <xacro:property name="kinematic_model" value="$(arg kinematic_model)"/>
+    <xacro:if value="${kinematic_model == 'body_assist'}">
+        <group name="arm_with_body">
+            <chain base_link="base_footprint" tip_link="arm0_hand"/>
+        </group>
+        <end_effector name="arm0_hand" parent_link="arm0_wrist_roll" group="arm_with_body"/>
+    </xacro:if>
+    <!-- Depending on the kinematic model, we have a different virtual joint to place spot in the environment -->
+    <xacro:unless value="${kinematic_model == 'none'}">
+        <virtual_joint name="spot_mobility_joint" child_link="base_footprint" parent_frame="spot_nav/map" type="planar"/>
+    </xacro:unless>
+    <xacro:if value="${kinematic_model == 'none'}">
+        <virtual_joint name="spot_mobility_joint" child_link="body" parent_frame="spot_nav/map" type="floating"/>
+    </xacro:if>
     <!--END EFFECTOR: Purpose: Represent information about an end effector.-->
-    <end_effector name="arm0_hand" parent_link="arm0_wrist_roll" group="arm_with_body"/>
     <end_effector name="arm0_hand" parent_link="arm0_wrist_roll" group="arm"/>
-    <!-- VIRTUAL JOINTS -->
-    <virtual_joint name="spot_mobility_joint" child_link="base_footprint" parent_frame="spot_nav/map" type="planar"/>
     <!--DISABLE COLLISIONS: By default it is assumed that any link of the robot could potentially come into collision with any other link in the robot. This tag disables collision checking between a specified pair of links. -->
     <disable_collisions link1="arm0_elbow_pitch" link2="arm0_elbow_roll" reason="Adjacent"/>

Commit message: disable collision between RL kit and body

File: spot_moveit_config/config/spot.srdf.xacro (robot description, xacro)
@@ -128,4 +128,7 @@
     <disable_collisions link1="arm0_base_link" link2="arm0_shoulder_yaw" reason="Adjacent"/>
     <disable_collisions link1="arm0_base_link" link2="body" reason="Adjacent"/>
+    <disable_collisions link1="body" link2="rl_kit_jetson_housing_box" reason="Adjacent"/>
+    <disable_collisions link1="body" link2="rl_kit_wire_housing_box" reason="Adjacent"/>
+    <disable_collisions link1="rl_kit_jetson_housing_box" link2="rl_kit_wire_housing_box" reason="Adjacent"/>
     <!-- Accessory collisions -->
     <xacro:arg name="has_eap"    default="False"/>

Commit message: add rl_kit_gpx_interface to non-colliding list

File: spot_moveit_config/config/spot.srdf.xacro (robot description, xacro)
@@ -130,5 +130,7 @@
     <disable_collisions link1="body" link2="rl_kit_jetson_housing_box" reason="Adjacent"/>
     <disable_collisions link1="body" link2="rl_kit_wire_housing_box" reason="Adjacent"/>
+    <disable_collisions link1="body" link2="rl_kit_gxp_interface" reason="Adjacent"/>
     <disable_collisions link1="rl_kit_jetson_housing_box" link2="rl_kit_wire_housing_box" reason="Adjacent"/>
+    <disable_collisions link1="rl_kit_gxp_interface" link2="rl_kit_wire_housing_box" reason="Adjacent" />
     <!-- Accessory collisions -->
     <xacro:arg name="has_eap"    default="False"/>

Commit message: disable collision between adjacent/fixed links

File: spot_moveit_config/config/spot.srdf.xacro (robot description, xacro)
@@ -133,4 +133,8 @@
     <disable_collisions link1="rl_kit_jetson_housing_box" link2="rl_kit_wire_housing_box" reason="Adjacent"/>
     <disable_collisions link1="rl_kit_gxp_interface" link2="rl_kit_wire_housing_box" reason="Adjacent" />
+    <disable_collisions link1="rl_kit_jetson_housing_box" link2="rl_kit_velodyne_mounting_plate" reason="Adjacent" />
+    <disable_collisions link1="velodyne" link2="velodyne_base_link" reason="Adjacent" />
+    <disable_collisions link1="velodyne" link2="velodyne_cage" reason="Adjacent" />
+    <disable_collisions link1="velodyne_base_link" link2="velodyne_cage" reason="Adjacent" />
     <!-- Accessory collisions -->
     <xacro:arg name="has_eap"    default="False"/>

Commit message: Removed hard-coded payload information and added unstow as predefined pose

File: spot_moveit_config/config/spot.srdf.xacro (robot description, xacro)
@@ -31,4 +31,13 @@
     <!--END EFFECTOR: Purpose: Represent information about an end effector.-->
     <end_effector name="arm0_hand" parent_link="arm0_wrist_roll" group="arm"/>
+    <!-- PRE-DEFINED STATES -->
+    <group_state name="unstowed" group="arm">
+        <joint name="arm0_shoulder_yaw" value="0.0"/>
+        <joint name="arm0_shoulder_pitch" value="-2.356"/>
+        <joint name="arm0_elbow_pitch" value="2.566"/>
+        <joint name="arm0_elbow_roll" value="0.07"/>
+        <joint name="arm0_wrist_pitch" value="-0.21"/>
+        <joint name="arm0_wrist_roll" value="-0.07"/>
+    </group_state>
     <!--DISABLE COLLISIONS: By default it is assumed that any link of the robot could potentially come into collision with any other link in the robot. This tag disables collision checking between a specified pair of links. -->
     <disable_collisions link1="arm0_elbow_pitch" link2="arm0_elbow_roll" reason="Adjacent"/>
@@ -133,8 +142,5 @@
     <disable_collisions link1="rl_kit_jetson_housing_box" link2="rl_kit_wire_housing_box" reason="Adjacent"/>
     <disable_collisions link1="rl_kit_gxp_interface" link2="rl_kit_wire_housing_box" reason="Adjacent" />
-    <disable_collisions link1="rl_kit_jetson_housing_box" link2="rl_kit_velodyne_mounting_plate" reason="Adjacent" />
     <disable_collisions link1="velodyne" link2="velodyne_base_link" reason="Adjacent" />
-    <disable_collisions link1="velodyne" link2="velodyne_cage" reason="Adjacent" />
-    <disable_collisions link1="velodyne_base_link" link2="velodyne_cage" reason="Adjacent" />
     <!-- Accessory collisions -->
     <xacro:arg name="has_eap"    default="False"/>

Commit message: add mobile_manipulation controllers and planning group

File: spot_moveit_config/config/spot.srdf.xacro (robot description, xacro)
@@ -22,4 +22,10 @@
         <end_effector name="arm0_hand" parent_link="arm0_wrist_roll" group="arm_with_body"/>
     </xacro:if>
+    <xacro:if value="${kinematic_model == 'mobile_manipulation'}">
+        <group name="mobile_body_and_arm">
+            <chain base_link="base_footprint" tip_link="arm0_fingers"/>
+        </group>
+        <end_effector name="arm0_hand" parent_link="arm0_wrist_roll" group="arm_with_body"/>
+    </xacro:if>
     <!-- Depending on the kinematic model, we have a different virtual joint to place spot in the environment -->
     <xacro:unless value="${kinematic_model == 'none'}">
@@ -29,4 +35,29 @@
         <virtual_joint name="spot_mobility_joint" child_link="body" parent_frame="spot_nav/map" type="floating"/>
     </xacro:if>
+    <!--GROUP STATES: Purpose: Define a named state for a particular group, in terms of joint values. This is useful to define states like 'folded arms'-->
+    <group_state name="namaste" group="mobile_body_and_arm">
+        <joint name="arm0_fingers" value="0"/>
+        <joint name="arm0_elbow_pitch" value="2.291"/>
+        <joint name="arm0_elbow_roll" value="0.0675"/>
+        <joint name="arm0_shoulder_pitch" value="-1.319"/>
+        <joint name="arm0_shoulder_yaw" value="-0.00415"/>
+        <joint name="arm0_wrist_pitch" value="-1.8326"/>
+        <joint name="arm0_wrist_roll" value="-0.0606"/>
+        <joint name="body_or" value="1.57"/>
+        <joint name="body_x" value="0.2"/>
+        <joint name="body_y" value="0.2"/>
+    </group_state>
+    <group_state name="home" group="mobile_body_and_arm">
+        <joint name="arm0_fingers" value="0"/>
+        <joint name="arm0_elbow_pitch" value="0"/>
+        <joint name="arm0_elbow_roll" value="0"/>
+        <joint name="arm0_shoulder_pitch" value="0"/>
+        <joint name="arm0_shoulder_yaw" value="0"/>
+        <joint name="arm0_wrist_pitch" value="0"/>
+        <joint name="arm0_wrist_roll" value="0"/>
+        <joint name="body_or" value="0"/>
+        <joint name="body_x" value="0"/>
+        <joint name="body_y" value="0"/>
+    </group_state>
     <!--END EFFECTOR: Purpose: Represent information about an end effector.-->
     <end_effector name="arm0_hand" parent_link="arm0_wrist_roll" group="arm"/>

Commit message: Added a collision free 'stowed' predefined state

File: spot_moveit_config/config/spot.srdf.xacro (robot description, xacro)
@@ -70,4 +70,12 @@
         <joint name="arm0_wrist_pitch" value="-0.21"/>
         <joint name="arm0_wrist_roll" value="-0.07"/>
+    </group_state>
+    <group_state name="stowed" group="arm">
+        <joint name="arm0_shoulder_yaw" value="0.0"/>
+        <joint name="arm0_shoulder_pitch" value="-3.14159265"/>
+        <joint name="arm0_elbow_pitch" value="3.12"/>
+        <joint name="arm0_elbow_roll" value="0.00"/>
+        <joint name="arm0_wrist_pitch" value="0.00"/>
+        <joint name="arm0_wrist_roll" value="0.00"/>
     </group_state>
     <!--DISABLE COLLISIONS: By default it is assumed that any link of the robot could potentially come into collision with any other link in the robot. This tag disables collision checking between a specified pair of links. -->

Commit message: Remove joint_limit error when planning

File: spot_moveit_config/config/spot.srdf.xacro (robot description, xacro)
@@ -11,6 +11,7 @@
     <!--SUBGROUPS: Groups can also be formed by referencing to already defined group names-->
     <group name="arm">
-        <chain base_link="arm0_base_link" tip_link="arm0_hand"/>
+        <chain base_link="arm0_base_link" tip_link="arm0_wrist_roll"/>
     </group>
+    <passive_joint name="arm0_fingers"/>
     <!-- Add the extra group if full body control is enabled -->
     <xacro:arg name="kinematic_model" default="none"/>
@@ -18,5 +19,5 @@
     <xacro:if value="${kinematic_model == 'body_assist'}">
         <group name="arm_with_body">
-            <chain base_link="base_footprint" tip_link="arm0_hand"/>
+            <chain base_link="base_footprint" tip_link="arm0_wrist_roll"/>
         </group>
         <end_effector name="arm0_hand" parent_link="arm0_wrist_roll" group="arm_with_body"/>
@@ -24,5 +25,5 @@
     <xacro:if value="${kinematic_model == 'mobile_manipulation'}">
         <group name="mobile_body_and_arm">
-            <chain base_link="base_footprint" tip_link="arm0_fingers"/>
+            <chain base_link="base_footprint" tip_link="arm0_wrist_roll"/>
         </group>
         <end_effector name="arm0_hand" parent_link="arm0_wrist_roll" group="arm_with_body"/>

Commit message: anchor mobile_manipulation virtual joint to odom and fix end effector group reference

File: spot_moveit_config/config/spot.srdf.xacro (robot description, xacro)
@@ -26,12 +26,15 @@
             <chain base_link="base_footprint" tip_link="arm0_fingers"/>
         </group>
-        <end_effector name="arm0_hand" parent_link="arm0_wrist_roll" group="arm_with_body"/>
+        <end_effector name="arm0_hand" parent_link="arm0_wrist_roll" group="mobile_body_and_arm"/>
     </xacro:if>
     <!-- Depending on the kinematic model, we have a different virtual joint to place spot in the environment -->
-    <xacro:unless value="${kinematic_model == 'none'}">
+    <xacro:if value="${kinematic_model == 'body_assist'}">
         <virtual_joint name="spot_mobility_joint" child_link="base_footprint" parent_frame="spot_nav/map" type="planar"/>
-    </xacro:unless>
+    </xacro:if>
     <xacro:if value="${kinematic_model == 'none'}">
         <virtual_joint name="spot_mobility_joint" child_link="body" parent_frame="spot_nav/map" type="floating"/>
+    </xacro:if>
+    <xacro:if value="${kinematic_model == 'mobile_manipulation'}">
+        <virtual_joint name="spot_mobility_joint" child_link="base_footprint" parent_frame="odom" type="floating"/>
     </xacro:if>
     <!--GROUP STATES: Purpose: Define a named state for a particular group, in terms of joint values. This is useful to define states like 'folded arms'-->
